File: NRF52840_Quiz_Remote/NRF52840_Quiz_Remote.kicad_pcb (KiCad board)
At the start: 2 copper layers, 66 x 152 mm, 32 parts, among them J1 NRF_LEFT, J2 NRF_RIGHT, SW1 ANSWER_A, SW2 ANSWER_B, SW3 ANSWER_C, SW4 ANSWER_D, SW5 SUBMIT, SW6 POWER, SW7 RESET

Commit message: sua B+/B-
Connections:
- J1 pad 1: /B+ -> GND
- J2 pad 1: /B- -> /B+
- J2 pad 3: Net-(J2-Pin_3) -> GND
- SW7 pad 1: Net-(J2-Pin_3) -> /RST
Routing:
- net /RST: track 0.00 -> 39.5 mm
- net Net-(J2-Pin_3): track 38.4 -> 0.00 mm
- net /B+: track 146.0 -> 166.5 mm
- net GND: track 321.8 -> 334.4 mm
