File: NRF52840_Quiz_Remote/NRF52840_Quiz_Remote.kicad_sch (KiCad schematic)
At the start: 28 parts, among them J1 NRF_LEFT, J2 NRF_RIGHT, SW1 ANSWER_A, SW2 ANSWER_B, SW3 ANSWER_C, SW4 ANSWER_D, SW5 SUBMIT, SW6 POWER, SW7 RESET

Commit message: web
Connections:
- net B- is gone; now on net B+: J2.1 (Pin_1)
- net B+: no longer J1.1 (Pin_1)
- net GND: now also J1.1 (Pin_1), J2.3 (Pin_3)
- net RST: now also SW7.1
Other:
- moved on the sheet: SW7
Changed lines of the file:
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@@
 	)
 	(junction
+		(at 168.91 91.44)
+		(diameter 0)
+		(color 0 0 0 0)
+	)
+	(junction
 		(at 22.86 66.04)
 		(diameter 0)
@@
 	)
 	(junction
+		(at 250.19 90.17)
+		(diameter 0)
+		(color 0 0 0 0)
+	)
+	(junction
 		(at 22.86 81.28)
 		(diameter 0)
@@
 	(wire
 		(pts
-			(xy 214.63 90.17) (xy 220.98 90.17)
+			(xy 214.63 90.17) (xy 231.14 90.17)
 		)
 		(stroke
@@
 	(wire
 		(pts
-			(xy 173.99 82.55) (xy 179.07 82.55)
-		)
-		(stroke
-			(width 0)
-			(type default)
-		)
-	)
-	(wire
-		(pts
 			(xy 29.21 149.86) (xy 29.21 161.29)
 		)
@@
 	(wire
 		(pts
-			(xy 242.57 87.63) (xy 248.92 87.63)
+			(xy 241.3 90.17) (xy 250.19 90.17)
 		)
 		(stroke
@@
 	(wire
 		(pts
-			(xy 248.92 87.63) (xy 248.92 91.44)
-		)
-		(stroke
-			(width 0)
-			(type default)
-		)
-	)
-	(wire
-		(pts
 			(xy 54.61 144.78) (xy 54.61 149.86)
 		)
@@
 	(wire
 		(pts
-			(xy 232.41 87.63) (xy 214.63 87.63)
+			(xy 168.91 82.55) (xy 179.07 82.55)
 		)
 		(stroke
@@
 	(wire
 		(pts
+			(xy 250.19 87.63) (xy 250.19 90.17)
+		)
+		(stroke
+			(width 0)
+			(type default)
+		)
+	)
+	(wire
+		(pts
 			(xy 76.2 57.15) (xy 76.2 81.28)
 		)
@@
 	(wire
 		(pts
+			(xy 168.91 91.44) (xy 173.99 91.44)
+		)
+		(stroke
+			(width 0)
+			(type default)
+		)
+	)
+	(wire
+		(pts
 			(xy 214.63 107.95) (xy 220.98 107.95)
 		)
@@
 	(wire
 		(pts
+			(xy 168.91 82.55) (xy 168.91 91.44)
+		)
+		(stroke
+			(width 0)
+			(type default)
+		)
+	)
+	(wire
+		(pts
 			(xy 29.21 179.07) (xy 54.61 179.07)
 		)
@@
 	(wire
 		(pts
+			(xy 214.63 87.63) (xy 250.19 87.63)
+		)
+		(stroke
+			(width 0)
+			(type default)
+		)
+	)
+	(wire
+		(pts
 			(xy 214.63 82.55) (xy 220.98 82.55)
 		)
@@
 	(wire
 		(pts
-			(xy 166.37 91.44) (xy 173.99 91.44)
+			(xy 166.37 91.44) (xy 168.91 91.44)
 		)
 		(stroke
@@
 		)
 	)
-	(label "B-"
+	(label "B+"
 		(at 220.98 82.55 0)
 		(effects
@@
 		)
 	)
+	(label "GND"
+		(at 220.98 87.63 0)
+		(effects
+			(font
+				(size 1.27 1.27)
+			)
+			(justify left bottom)
+		)
+	)
 	(label "P0.02"
 		(at 220.98 100.33 0)
@@
 		)
 	)
-	(label "B+"
-		(at 173.99 82.55 0)
-		(effects
-			(font
-				(size 1.27 1.27)
-			)
-			(justify left bottom)
-		)
-	)
 	(label "P1.13"
 		(at 220.98 105.41 0)
@@
 	(symbol
 		(lib_id "Switch:SW_Push")
-		(at 237.49 87.63 0)
+		(at 236.22 90.17 0)
 		(unit 1)
 		(body_style 1)
@@
 		(fields_autoplaced yes)
 		(property "Reference" "SW7"
-			(at 237.49 80.01 0)
+			(at 236.22 82.55 0)
 			(show_name no)
 			(do_not_autoplace no)
@@
 		)
 		(property "Value" "RESET"
-			(at 237.49 82.55 0)
+			(at 236.22 85.09 0)
 			(show_name no)
 			(do_not_autoplace no)
@@
 		)
 		(property "Footprint" "Button_Switch_THT:SW_PUSH_6mm_H4.3mm"
-			(at 237.49 82.55 0)
+			(at 236.22 85.09 0)
 			(hide yes)
 			(show_name no)
@@
 		)
 		(property "Datasheet" ""
-			(at 237.49 82.55 0)
+			(at 236.22 85.09 0)
 			(hide yes)
 			(show_name no)
@@
 		)
 		(property "Description" "Push button switch, generic, two pins"
-			(at 237.49 87.63 0)
+			(at 236.22 90.17 0)
 			(hide yes)
 			(show_name no)
@@
 	(symbol
 		(lib_id "power:GND")
-		(at 248.92 91.44 0)
+		(at 250.19 90.17 0)
 		(unit 1)
 		(body_style 1)
@@
 		(fields_autoplaced yes)
 		(property "Reference" "#PWR02"
-			(at 248.92 97.79 0)
+			(at 250.19 96.52 0)
 			(hide yes)
 			(show_name no)
@@
 		)
 		(property "Value" "GND"
-			(at 248.92 96.52 0)
+			(at 250.19 95.25 0)
 			(show_name no)
 			(do_not_autoplace no)
@@
 		)
 		(property "Footprint" ""
-			(at 248.92 91.44 0)
+			(at 250.19 90.17 0)
 			(hide yes)
 			(show_name no)
@@
 		)
 		(property "Datasheet" ""
-			(at 248.92 91.44 0)
+			(at 250.19 90.17 0)
 			(hide yes)
 			(show_name no)
@@
 		)
 		(property "Description" "Power symbol creates a global label with name \"GND\" , ground"
-			(at 248.92 91.44 0)
+			(at 250.19 90.17 0)
 			(hide yes)
 			(show_name no)
